File: Bald DAC Wing.kicad_pcb (KiCad board)
At the start: 4 copper layers, 62.2 x 46.5 mm, 46 parts, among them J1 PWR, J10 Ctrl Debug, J11 BNC_B, J13 Feather Debug, J2 DAC_A_Out, J3 DAC_B_Out, J4 BNC_Z, J5 Z_Out, J6 Feather, J7 Data Debug Low, J8 BNC_A, J9 Data Debug High, U1 AD5447, U2 AD8065ARTZ, U3 AD8065ARTZ, U4 74LVC574APWR, U5 74LVC574APWR, U6 74LVC1G04, U7 REF3425

Commit message: gonna try and submit.
Parts:
- added REF**: KiCad-Logo2_8mm_SilkScreen, Symbol:KiCad-Logo2_8mm_SilkScreen, B.Cu at (126.2, 91.9)
- added kibuzzard-6AB05686: G***, kibuzzard-6AB05686, F.Cu at (125.9, 73.0)
- added kibuzzard-6AB056B3: G***, kibuzzard-6AB056B3, F.Cu at (140.6, 111.8)
Other:
- board text added: "0"
- board text added: "1"
- board text added: "10"
- board text added: "11"
- board text added: "2"
- board text added: "3"
- board text added: "4"
- board text added: "5"
- board text added: "6"
- board text added: "7"
- board text added: "8"
- board text added: "9"
- board text added: "AB"
- board text added: "D0"
- board text added: "D1"
- board text added: "D2"
- board text added: "D3"
- board text added: "D4"
- board text added: "D5"
- board text added: "GND"
- board text added: "H"
- board text added: "L"
- board text added: "LCLK"
- board text added: "LOE"
- board text added: "OUTA"
- board text added: "OUTB"
- board text added: "OUTZ"
- board text added: "R_EN"
- board text added: "Z"
- board text added: "~{CS}"
